File: kicad/display.kicad_sch (KiCad schematic)
At the start: 0 parts

Commit message: gain, meter and display sheets
Parts:
- added U8: TCA9548AMRGER, Package_DFN_QFN:Texas_RGE0024C_VQFN-24-1EP_4x4mm_P0.5mm_EP2.1x2.1mm, symbol Interface_Expansion:TCA9548AMRGER
- added oled1, oled2, oled3, oled4, oled5, oled6, oled7, oled8: ~, symbol mixer:ssd1306
Connections:
- new net: U8.2 (SC0), oled1.3 (SCL)
- new net: U8.1 (SD0), oled1.4 (SCA)
- new net: U8.13 (SC5), oled6.3 (SCL)
- new net: U8.12 (SD5), oled6.4 (SCA)
- new net: U8.17 (SC7), oled8.3 (SCL)
- new net: U8.16 (SD7), oled8.4 (SCA)
- new net: U8.4 (SC1), oled2.3 (SCL)
- new net: U8.3 (SD1), oled2.4 (SCA)
- new net: U8.8 (SC3), oled4.3 (SCL)
- new net: U8.7 (SD3), oled4.4 (SCA)
- new net: U8.6 (SC2), oled3.3 (SCL)
- new net: U8.5 (SD2), oled3.4 (SCA)
- new net: U8.11 (SC4), oled5.3 (SCL)
- new net: U8.10 (SD4), oled5.4 (SCA)
- new net: U8.14 (SD6), oled7.4 (SCA)
- new net: U8.15 (SC6), oled7.3 (SCL)
- new net +5V: U8.21 (VCC), oled1.2 (VCC), oled2.2 (VCC), oled3.2 (VCC), oled4.2 (VCC), oled5.2 (VCC), oled6.2 (VCC), oled7.2 (VCC), oled8.2 (VCC)
- new net A0: U8.22 (A0)
- new net A1: U8.23 (A1)
- new net A2: U8.18 (A2)
- new net GND: U8.9 (GND), oled1.1 (GND), oled2.1 (GND), oled3.1 (GND), oled4.1 (GND), oled5.1 (GND), oled6.1 (GND), oled7.1 (GND), oled8.1 (GND)
- new net SCL: U8.19 (SCL)
- new net SDA: U8.20 (SDA)
