File: kicad/mixer.kicad_pcb (KiCad board)
At the start: 2 copper layers, 72 parts, among them U10 GREEN_LOWER, U11 RED, U12 YELLOW, U13 CD74HC4067M96, U4 MAX7219, U6 CD74HC4067M, U7 TCA9548APWR, U9 GREEN_UPPER

Commit message: pcb routing 1
Parts:
- U10, U11, U12, U9: moved to B.Cu
- moved C2 272.5 mm to (30.2, 84.8)
- moved R4 272.5 mm to (27.9, 91.8)
- moved C1 271.9 mm to (28.2, 16.5)
- moved R3 271.9 mm to (25.9, 23.5)
- moved U11 119.1 mm to (314.8, 46.4), turned to 180 degrees
- moved U10 104.2 mm to (60.4, 95.8), turned to 180 degrees
- moved U9 89.5 mm to (314.8, 95.5), turned to 180 degrees
- moved C8 64.0 mm to (391.9, 112.5)
- moved U13 64.0 mm to (379.0, 111.8)
- moved U12 29.9 mm to (58.8, 46.0), turned to 180 degrees
- moved C12 26.1 mm to (338.5, 85.0)
- moved R1 26.1 mm to (336.2, 92.5)
- moved C13 8.27 mm to (341.5, 19.5)
- moved R2 8.27 mm to (339.2, 26.5)
- moved C9 4.96 mm to (334.8, 131.9)
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Connections:
- BAR10 pad 1: Net-(U9-DIG_1) -> Net-(U9-DIG_4)
- BAR10 pad 10: Net-(U10-DIG_1) -> Net-(U10-DIG_4)
- BAR10 pad 2: Net-(U9-DIG_1) -> Net-(U9-DIG_4)
- BAR10 pad 3: Net-(U9-DIG_1) -> Net-(U9-DIG_4)
- BAR10 pad 4: Net-(U9-DIG_1) -> Net-(U9-DIG_4)
- BAR10 pad 5: Net-(U9-DIG_1) -> Net-(U9-DIG_4)
- BAR10 pad 6: Net-(U10-DIG_1) -> Net-(U10-DIG_4)
- BAR10 pad 7: Net-(U10-DIG_1) -> Net-(U10-DIG_4)
- BAR10 pad 8: Net-(U10-DIG_1) -> Net-(U10-DIG_4)
- BAR10 pad 9: Net-(U10-DIG_1) -> Net-(U10-DIG_4)
- BAR11 pad 1: Net-(U9-DIG_2) -> Net-(U9-DIG_6)
- BAR11 pad 10: Net-(U10-DIG_2) -> Net-(U10-DIG_6)
- BAR11 pad 2: Net-(U9-DIG_2) -> Net-(U9-DIG_6)
- BAR11 pad 3: Net-(U9-DIG_2) -> Net-(U9-DIG_6)
- BAR11 pad 4: Net-(U9-DIG_2) -> Net-(U9-DIG_6)
- BAR11 pad 5: Net-(U9-DIG_2) -> Net-(U9-DIG_6)
- BAR11 pad 6: Net-(U10-DIG_2) -> Net-(U10-DIG_6)
- BAR11 pad 7: Net-(U10-DIG_2) -> Net-(U10-DIG_6)
- BAR11 pad 8: Net-(U10-DIG_2) -> Net-(U10-DIG_6)
- BAR11 pad 9: Net-(U10-DIG_2) -> Net-(U10-DIG_6)
- BAR12 pad 1: Net-(U9-DIG_3) -> Net-(U9-DIG_2)
- BAR12 pad 10: Net-(U10-DIG_3) -> Net-(U10-DIG_2)
- BAR12 pad 2: Net-(U9-DIG_3) -> Net-(U9-DIG_2)
- BAR12 pad 3: Net-(U9-DIG_3) -> Net-(U9-DIG_2)
- BAR12 pad 4: Net-(U9-DIG_3) -> Net-(U9-DIG_2)
- BAR12 pad 5: Net-(U9-DIG_3) -> Net-(U9-DIG_2)
- BAR12 pad 6: Net-(U10-DIG_3) -> Net-(U10-DIG_2)
- BAR12 pad 7: Net-(U10-DIG_3) -> Net-(U10-DIG_2)
- BAR12 pad 8: Net-(U10-DIG_3) -> Net-(U10-DIG_2)
- BAR12 pad 9: Net-(U10-DIG_3) -> Net-(U10-DIG_2)
- BAR13 pad 1: Net-(U9-DIG_4) -> Net-(U9-DIG_3)
- BAR13 pad 10: Net-(U10-DIG_4) -> Net-(U10-DIG_3)
- BAR13 pad 2: Net-(U9-DIG_4) -> Net-(U9-DIG_3)
- BAR13 pad 3: Net-(U9-DIG_4) -> Net-(U9-DIG_3)
- BAR13 pad 4: Net-(U9-DIG_4) -> Net-(U9-DIG_3)
- BAR13 pad 5: Net-(U9-DIG_4) -> Net-(U9-DIG_3)
- BAR13 pad 6: Net-(U10-DIG_4) -> Net-(U10-DIG_3)
- BAR13 pad 7: Net-(U10-DIG_4) -> Net-(U10-DIG_3)
- BAR13 pad 8: Net-(U10-DIG_4) -> Net-(U10-DIG_3)
- BAR13 pad 9: Net-(U10-DIG_4) -> Net-(U10-DIG_3)
- BAR14 pad 1: Net-(U9-DIG_5) -> Net-(U9-DIG_7)
- BAR14 pad 10: Net-(U10-DIG_5) -> Net-(U10-DIG_7)
- BAR14 pad 2: Net-(U9-DIG_5) -> Net-(U9-DIG_7)
- BAR14 pad 3: Net-(U9-DIG_5) -> Net-(U9-DIG_7)
- BAR14 pad 4: Net-(U9-DIG_5) -> Net-(U9-DIG_7)
- BAR14 pad 5: Net-(U9-DIG_5) -> Net-(U9-DIG_7)
- BAR14 pad 6: Net-(U10-DIG_5) -> Net-(U10-DIG_7)
- BAR14 pad 7: Net-(U10-DIG_5) -> Net-(U10-DIG_7)
- BAR14 pad 8: Net-(U10-DIG_5) -> Net-(U10-DIG_7)
- BAR14 pad 9: Net-(U10-DIG_5) -> Net-(U10-DIG_7)
- BAR15 pad 1: Net-(U9-DIG_6) -> Net-(U9-DIG_5)
- BAR15 pad 10: Net-(U10-DIG_6) -> Net-(U10-DIG_5)
- BAR15 pad 2: Net-(U9-DIG_6) -> Net-(U9-DIG_5)
- BAR15 pad 3: Net-(U9-DIG_6) -> Net-(U9-DIG_5)
- BAR15 pad 4: Net-(U9-DIG_6) -> Net-(U9-DIG_5)
- BAR15 pad 5: Net-(U9-DIG_6) -> Net-(U9-DIG_5)
- BAR15 pad 6: Net-(U10-DIG_6) -> Net-(U10-DIG_5)
- BAR15 pad 7: Net-(U10-DIG_6) -> Net-(U10-DIG_5)
- BAR15 pad 8: Net-(U10-DIG_6) -> Net-(U10-DIG_5)
- BAR15 pad 9: Net-(U10-DIG_6) -> Net-(U10-DIG_5)
- BAR16 pad 1: Net-(U9-DIG_7) -> Net-(U9-DIG_1)
- BAR16 pad 10: Net-(U10-DIG_7) -> Net-(U10-DIG_1)
- BAR16 pad 2: Net-(U9-DIG_7) -> Net-(U9-DIG_1)
- BAR16 pad 3: Net-(U9-DIG_7) -> Net-(U9-DIG_1)
- BAR16 pad 4: Net-(U9-DIG_7) -> Net-(U9-DIG_1)
- BAR16 pad 5: Net-(U9-DIG_7) -> Net-(U9-DIG_1)
- BAR16 pad 6: Net-(U10-DIG_7) -> Net-(U10-DIG_1)
- BAR16 pad 7: Net-(U10-DIG_7) -> Net-(U10-DIG_1)
- BAR16 pad 8: Net-(U10-DIG_7) -> Net-(U10-DIG_1)
- BAR16 pad 9: Net-(U10-DIG_7) -> Net-(U10-DIG_1)
- BAR2 pad 1: Net-(U11-DIG_1) -> Net-(U11-DIG_4)
- BAR2 pad 10: Net-(U12-DIG_1) -> Net-(U12-DIG_4)
- BAR2 pad 2: Net-(U11-DIG_1) -> Net-(U11-DIG_4)
- BAR2 pad 3: Net-(U11-DIG_1) -> Net-(U11-DIG_4)
- BAR2 pad 4: Net-(U11-DIG_1) -> Net-(U11-DIG_4)
- BAR2 pad 5: Net-(U11-DIG_1) -> Net-(U11-DIG_4)
- BAR2 pad 6: Net-(U12-DIG_1) -> Net-(U12-DIG_4)
- BAR2 pad 7: Net-(U12-DIG_1) -> Net-(U12-DIG_4)
- BAR2 pad 8: Net-(U12-DIG_1) -> Net-(U12-DIG_4)
- BAR2 pad 9: Net-(U12-DIG_1) -> Net-(U12-DIG_4)
- BAR3 pad 1: Net-(U11-DIG_2) -> Net-(U11-DIG_6)
- BAR3 pad 10: Net-(U12-DIG_2) -> Net-(U12-DIG_6)
- BAR3 pad 2: Net-(U11-DIG_2) -> Net-(U11-DIG_6)
- BAR3 pad 3: Net-(U11-DIG_2) -> Net-(U11-DIG_6)
- BAR3 pad 4: Net-(U11-DIG_2) -> Net-(U11-DIG_6)
- BAR3 pad 5: Net-(U11-DIG_2) -> Net-(U11-DIG_6)
- BAR3 pad 6: Net-(U12-DIG_2) -> Net-(U12-DIG_6)
- BAR3 pad 7: Net-(U12-DIG_2) -> Net-(U12-DIG_6)
- BAR3 pad 8: Net-(U12-DIG_2) -> Net-(U12-DIG_6)
- BAR3 pad 9: Net-(U12-DIG_2) -> Net-(U12-DIG_6)
- BAR4 pad 1: Net-(U11-DIG_3) -> Net-(U11-DIG_2)
- BAR4 pad 10: Net-(U12-DIG_3) -> Net-(U12-DIG_2)
- BAR4 pad 2: Net-(U11-DIG_3) -> Net-(U11-DIG_2)
- BAR4 pad 3: Net-(U11-DIG_3) -> Net-(U11-DIG_2)
- BAR4 pad 4: Net-(U11-DIG_3) -> Net-(U11-DIG_2)
- BAR4 pad 5: Net-(U11-DIG_3) -> Net-(U11-DIG_2)
- BAR4 pad 6: Net-(U12-DIG_3) -> Net-(U12-DIG_2)
- BAR4 pad 7: Net-(U12-DIG_3) -> Net-(U12-DIG_2)
- BAR4 pad 8: Net-(U12-DIG_3) -> Net-(U12-DIG_2)
- BAR4 pad 9: Net-(U12-DIG_3) -> Net-(U12-DIG_2)
- BAR5 pad 1: Net-(U11-DIG_4) -> Net-(U11-DIG_3)
- BAR5 pad 10: Net-(U12-DIG_4) -> Net-(U12-DIG_3)
- BAR5 pad 2: Net-(U11-DIG_4) -> Net-(U11-DIG_3)
- BAR5 pad 3: Net-(U11-DIG_4) -> Net-(U11-DIG_3)
- BAR5 pad 4: Net-(U11-DIG_4) -> Net-(U11-DIG_3)
- BAR5 pad 5: Net-(U11-DIG_4) -> Net-(U11-DIG_3)
- BAR5 pad 6: Net-(U12-DIG_4) -> Net-(U12-DIG_3)
- BAR5 pad 7: Net-(U12-DIG_4) -> Net-(U12-DIG_3)
- BAR5 pad 8: Net-(U12-DIG_4) -> Net-(U12-DIG_3)
- BAR5 pad 9: Net-(U12-DIG_4) -> Net-(U12-DIG_3)
- BAR6 pad 1: Net-(U11-DIG_5) -> Net-(U11-DIG_7)
- BAR6 pad 10: Net-(U12-DIG_5) -> Net-(U12-DIG_7)
- BAR6 pad 2: Net-(U11-DIG_5) -> Net-(U11-DIG_7)
- BAR6 pad 3: Net-(U11-DIG_5) -> Net-(U11-DIG_7)
- BAR6 pad 4: Net-(U11-DIG_5) -> Net-(U11-DIG_7)
- BAR6 pad 5: Net-(U11-DIG_5) -> Net-(U11-DIG_7)
- BAR6 pad 6: Net-(U12-DIG_5) -> Net-(U12-DIG_7)
- BAR6 pad 7: Net-(U12-DIG_5) -> Net-(U12-DIG_7)
- BAR6 pad 8: Net-(U12-DIG_5) -> Net-(U12-DIG_7)
- BAR6 pad 9: Net-(U12-DIG_5) -> Net-(U12-DIG_7)
- BAR7 pad 1: Net-(U11-DIG_6) -> Net-(U11-DIG_5)
- BAR7 pad 10: Net-(U12-DIG_6) -> Net-(U12-DIG_5)
- BAR7 pad 2: Net-(U11-DIG_6) -> Net-(U11-DIG_5)
- BAR7 pad 3: Net-(U11-DIG_6) -> Net-(U11-DIG_5)
- BAR7 pad 4: Net-(U11-DIG_6) -> Net-(U11-DIG_5)
- BAR7 pad 5: Net-(U11-DIG_6) -> Net-(U11-DIG_5)
- BAR7 pad 6: Net-(U12-DIG_6) -> Net-(U12-DIG_5)
- BAR7 pad 7: Net-(U12-DIG_6) -> Net-(U12-DIG_5)
- BAR7 pad 8: Net-(U12-DIG_6) -> Net-(U12-DIG_5)
- BAR7 pad 9: Net-(U12-DIG_6) -> Net-(U12-DIG_5)
- BAR8 pad 1: Net-(U11-DIG_7) -> Net-(U11-DIG_1)
- BAR8 pad 10: Net-(U12-DIG_7) -> Net-(U12-DIG_1)
- BAR8 pad 2: Net-(U11-DIG_7) -> Net-(U11-DIG_1)
- BAR8 pad 3: Net-(U11-DIG_7) -> Net-(U11-DIG_1)
- BAR8 pad 4: Net-(U11-DIG_7) -> Net-(U11-DIG_1)
- BAR8 pad 5: Net-(U11-DIG_7) -> Net-(U11-DIG_1)
- BAR8 pad 6: Net-(U12-DIG_7) -> Net-(U12-DIG_1)
- BAR8 pad 7: Net-(U12-DIG_7) -> Net-(U12-DIG_1)
- BAR8 pad 8: Net-(U12-DIG_7) -> Net-(U12-DIG_1)
- BAR8 pad 9: Net-(U12-DIG_7) -> Net-(U12-DIG_1)
Routing:
- net Net-(U9-SEG_A): track 0.00 -> 552.1 mm, vias 0 -> 8
- net Net-(U9-SEG_B): track 0.00 -> 503.1 mm, vias 0 -> 8
- net Net-(U10-SEG_A): track 0.00 -> 473.7 mm, vias 0 -> 8
- net Net-(U9-SEG_C): track 0.00 -> 447.6 mm, vias 0 -> 8
- net Net-(U10-SEG_B): track 0.00 -> 433.9 mm, vias 0 -> 8
- net Net-(U9-SEG_D): track 0.00 -> 390.3 mm, vias 0 -> 8
- net Net-(U10-SEG_C): track 0.00 -> 390.1 mm, vias 0 -> 8
- net Net-(U9-SEG_E): track 0.00 -> 362.6 mm, vias 0 -> 8
- net Net-(U10-SEG_D): track 0.00 -> 357.4 mm, vias 0 -> 8
- net Net-(U9-DIG_0): track 0.00 -> 324.7 mm, vias 0 -> 5
- net Net-(U10-SEG_E): track 0.00 -> 317.1 mm, vias 0 -> 8
- net Net-(U9-DIG_4): track 0.00 -> 290.7 mm, vias 0 -> 5
- net Net-(U9-DIG_6): track 0.00 -> 265.9 mm, vias 0 -> 5
- net Net-(U10-DIG_1): track 0.00 -> 257.2 mm, vias 0 -> 5
- net Net-(U9-DIG_2): track 0.00 -> 245.7 mm, vias 0 -> 5
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Other:
- copper layers 2 -> 4

Commit message: pcb routing 2
Parts:
- moved U13 66.0 mm to (313.5, 119.5), turned to 90 degrees
- moved C9 38.0 mm to (297.2, 126.5)
- moved C1 28.6 mm to (26.2, 45.0)
- moved R3 28.6 mm to (23.9, 52.0)
- moved C13 27.0 mm to (340.0, 46.5)
- moved R2 27.0 mm to (337.7, 53.5)
- moved U9 16.8 mm to (317.0, 78.9)
- moved U4 6.61 mm to (313.9, 134.9)
- moved U11 4.62 mm to (315.6, 41.8)
- moved U12 0.72 mm to (59.5, 45.8)
- moved BAR14 0.26 mm to (221.3, 71.5)
- moved BAR15 0.26 mm to (249.3, 71.5)
- moved BAR10 0.26 mm to (109.3, 71.5)
- moved BAR1 0.19 mm to (81.3, 45.5)
- moved BAR11 0.18 mm to (137.3, 71.5)
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Connections:
- SW1 pad 1: (no net) -> Net-(SW1-B)
- SW1 pad 2: (no net) -> Net-(SW1-C)
- SW1 pad 3: (no net) -> GND
- SW2 pad 1: (no net) -> Net-(SW2-C)
- SW2 pad 2: (no net) -> Net-(SW2-B)
- SW2 pad 3: (no net) -> GND
- SW3 pad 1: (no net) -> Net-(SW3-A)
- SW3 pad 2: (no net) -> Net-(SW3-B)
- SW3 pad 3: (no net) -> GND
- SW4 pad 1: (no net) -> Net-(SW4-C)
- SW4 pad 2: (no net) -> Net-(SW4-B)
- SW4 pad 3: (no net) -> GND
- SW5 pad 1: (no net) -> Net-(SW5-A)
- SW5 pad 2: (no net) -> Net-(SW5-C)
- SW5 pad 3: (no net) -> GND
- SW6 pad 1: (no net) -> Net-(SW6-C)
- SW6 pad 2: (no net) -> Net-(SW6-B)
- SW6 pad 3: (no net) -> GND
- SW7 pad 1: (no net) -> Net-(SW7-C)
- SW7 pad 2: (no net) -> Net-(SW7-B)
- SW7 pad 3: (no net) -> GND
- SW8 pad 1: (no net) -> Net-(SW8-B)
- SW8 pad 2: (no net) -> Net-(SW8-A)
- SW8 pad 3: (no net) -> GND
- U13 pad 16: Net-(SW8-C) -> Net-(SW8-A)
- U13 pad 17: Net-(SW8-A) -> Net-(SW8-B)
- U13 pad 18: Net-(SW7-C) -> Net-(SW7-B)
- U13 pad 19: Net-(SW7-A) -> Net-(SW7-C)
- U13 pad 2: Net-(SW4-C) -> Net-(SW4-B)
- U13 pad 20: Net-(SW6-C) -> Net-(SW6-B)
- U13 pad 21: Net-(SW6-A) -> Net-(SW6-C)
- U13 pad 3: Net-(SW4-A) -> Net-(SW4-C)
- U13 pad 4: Net-(SW3-C) -> Net-(SW3-B)
- U13 pad 6: Net-(SW2-C) -> Net-(SW2-B)
- U13 pad 7: Net-(SW2-A) -> Net-(SW2-C)
- U13 pad 9: Net-(SW1-A) -> Net-(SW1-B)
Routing:
- net (no net): track 0.00 -> 479.3 mm
- net Net-(U9-SEG_A): track 552.1 -> 237.6 mm, vias 8 -> 7
- net Net-(U10-SEG_A): track 473.7 -> 180.9 mm
- net Net-(U10-SEG_D): track 357.4 -> 65.4 mm
- net Net-(U10-SEG_B): track 433.9 -> 142.2 mm
- net Net-(U10-SEG_C): track 390.1 -> 104.5 mm
- net Net-(U12-SEG_E): track 0.00 -> 281.7 mm, vias 0 -> 7
- net Net-(U10-SEG_E): track 317.1 -> 35.4 mm
- net Net-(U9-SEG_B): track 503.1 -> 234.9 mm
- net Net-(U9-SEG_C): track 447.6 -> 197.2 mm
- net Net-(U12-SEG_D): track 0.00 -> 245.8 mm, vias 0 -> 6
- net Net-(U9-SEG_E): track 362.6 -> 124.5 mm
- net Net-(U9-SEG_D): track 390.3 -> 158.3 mm
- net Net-(U12-SEG_C): track 0.00 -> 206.6 mm, vias 0 -> 6
- net Net-(U12-DIG_0): track 24.4 -> 229.3 mm, vias 5 -> 0
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Other:
- board text added: "${REFERENCE}"

Commit message: kicad - pcb routing
Parts:
-  1: moved to B.Cu
-  11: moved to B.Cu
-  111: moved to B.Cu
- C1, C10, C11, C12, C13, C2, C8, C9, R1, R2, R3, R4, R5, U13, U4, U6, U7: moved to B.Cu
- moved C1 320.7 mm to (307.2, 199.5), turned to 180 degrees
- moved C2 292.9 mm to (306.8, 181.2), turned to 180 degrees
- moved R2 257.8 mm to (116.0, 185.2), turned to -90 degrees
- moved R4 234.8 mm to (244.0, 183.7), turned to -90 degrees
- moved R3 221.9 mm to (201.8, 184.7), turned to -90 degrees
- moved U9 219.4 mm to (125.6, 186.1), turned to -90 degrees
- moved U12 207.3 mm to (212.2, 186.1), turned to -90 degrees
- moved U11 205.6 mm to (169.0, 186.0), turned to -90 degrees
- moved R1 200.3 mm to (158.5, 184.9), turned to -90 degrees
- moved C10 191.0 mm to (120.8, 186.2), turned to -90 degrees
- moved C11 174.3 mm to (163.8, 194.0), turned to 90 degrees
- moved C12 134.9 mm to (248.8, 185.8), turned to -90 degrees
- moved C8 127.5 mm to (283.2, 179.0), turned to 180 degrees
- moved  111 126.4 mm to (302.0, 92.3)
- moved  1 110.5 mm to (313.4, 145.4)
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Routing:
- net GND: track 0.02 -> 934.2 mm
- net Net-(U11-SEG_A): track 29.7 -> 822.3 mm, vias 6 -> 8
- net Net-(U11-SEG_B): track 61.2 -> 800.4 mm, vias 7 -> 8
- net Net-(U11-SEG_C): track 97.4 -> 784.8 mm, vias 6 -> 8
- net Net-(U11-SEG_D): track 136.5 -> 763.7 mm, vias 6 -> 8
- net Net-(U11-SEG_E): track 173.8 -> 738.8 mm, vias 6 -> 8
- net Net-(U12-SEG_A): track 135.4 -> 679.6 mm, vias 7 -> 8
- net Net-(U12-SEG_B): track 169.2 -> 659.0 mm, vias 6 -> 8
- net (no net): track 479.3 -> 0.00 mm
- net Net-(U12-SEG_C): track 206.6 -> 644.0 mm, vias 6 -> 8
- net Net-(U12-SEG_D): track 245.8 -> 623.5 mm, vias 6 -> 8
- net Net-(U9-SEG_E): track 124.5 -> 494.5 mm
- net Net-(U9-SEG_A): track 237.6 -> 596.9 mm, vias 7 -> 8
- net Net-(U9-SEG_D): track 158.3 -> 516.3 mm
- net Net-(U9-SEG_C): track 197.2 -> 542.8 mm
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Other:
- board text removed: "${REFERENCE}"

Commit message: esp idf testing
Parts:
- removed  1: HEADER-10, Connector_PinHeader_2.54mm:PinHeader_1x10_P2.54mm_Horizontal
- removed  11: HEADER-10, Connector_PinHeader_2.54mm:PinHeader_1x10_P2.54mm_Horizontal
- removed  111: HEADER-10, Connector_PinHeader_2.54mm:PinHeader_1x10_P2.54mm_Horizontal
- removed BAR1, BAR10, BAR11, BAR12, BAR13, BAR14, BAR15, BAR16, BAR2, BAR3, BAR4, BAR5, BAR6, BAR7, BAR8, BAR9: HDSP-4832_2, Display:HDSP-4832
- removed C1, C10, C11, C12, C13, C2, C8, C9: 100nF, Capacitor_THT:C_Axial_L5.1mm_D3.1mm_P7.50mm_Horizontal
- removed R1, R2, R3, R4, R5: R, Resistor_THT:R_Axial_DIN0207_L6.3mm_D2.5mm_P10.16mm_Horizontal
- removed SW1, SW2, SW3, SW4, SW5, SW6, SW7, SW8: ~, mixer:RotaryEncoder
- removed U10: GREEN_LOWER, Package_DIP:DIP-24_W7.62mm_Socket
- removed U11: RED, Package_DIP:DIP-24_W7.62mm_Socket
- removed U12: YELLOW, Package_DIP:DIP-24_W7.62mm_Socket
- removed U13: CD74HC4067M96, digikey-footprints:SOIC-24_W7.50mm
- removed U7: TCA9548APWR, digikey-footprints:TSSOP-24_W4.40mm
- removed U9: GREEN_UPPER, Package_DIP:DIP-24_W7.62mm_Socket
- removed mute10, mute11, mute12, mute13, mute14, mute15, mute16, mute9, solo3, solo4, solo5, solo6, solo7, solo8: SW_SPST_LED, mixer:SW_SPST_LED_9mm
- removed oled3, oled4, oled5, oled6, oled7, oled8: ~, mixer:oled
- added LowerLED1: HDSP-4832_2, Display:HDSP-4832, F.Cu at (82.1, 129.7)
- added LowerLED2: HDSP-4832_2, Display:HDSP-4832, F.Cu at (109.9, 129.8)
- added SW10: ~, mixer:RotaryEncoder, F.Cu at (113.8, 87.5)
- added SW9: ~, mixer:RotaryEncoder, F.Cu at (86.0, 87.8)
- added UpperLED1: HDSP-4832_2, Display:HDSP-4832, F.Cu at (82.1, 103.6)
- added UpperLED2: HDSP-4832_2, Display:HDSP-4832, F.Cu at (109.9, 103.7)
- added mute1: SW_SPST_LED, mixer:SW_SPST_LED_9mm, F.Cu at (86.0, 186.0)
- added mute2: SW_SPST_LED, mixer:SW_SPST_LED_9mm, F.Cu at (114.0, 186.0)
- U4: value MAX7219 -> MCP23017_SP; footprint Package_DIP:DIP-24_W7.62mm_Socket -> Package_DIP:DIP-28_W7.62mm
- U6: value CD74HC4067M -> MAX7219; footprint Package_SO:SOIC-24W_7.5x15.4mm_P1.27mm -> Package_DIP:DIP-24_W7.62mm
- moved U6 208.0 mm to (95.8, 131.5), turned to 0 degrees
- moved U4 157.2 mm to (95.9, 189.1), turned to 0 degrees
- moved solo1 25.3 mm to (86.0, 164.2)
- moved solo2 25.3 mm to (113.8, 164.2)
- moved oled1 25.1 mm to (86.0, 212.0)
- moved oled2 25.1 mm to (114.0, 212.0)
Connections:
- U4 pad 1: /buttons/DIN -> Net-(U4-GPB0)
- U4 pad 10: unconnected-(U4-DIG_5-Pad10) -> Earth
- U4 pad 11: Net-(U4-DIG_1) -> unconnected-(U4-NC-Pad11)
- U4 pad 12: /buttons/LOAD -> Net-(J3-Pin_1)
- U4 pad 13: /buttons/CLK -> Net-(J1-Pin_1)
- U4 pad 14: Net-(U4-SEG_A) -> unconnected-(U4-NC-Pad14)
- U4 pad 15: Net-(U4-SEG_F) -> unconnected-(U4-A0-Pad15)
- U4 pad 16: Net-(U4-SEG_B) -> unconnected-(U4-A1-Pad16)
- U4 pad 17: Net-(U4-SEG_G) -> unconnected-(U4-A2-Pad17)
- U4 pad 18: Net-(U4-ISET) -> unconnected-(U4-~{RESET}-Pad18)
- U4 pad 19: +5V -> unconnected-(U4-INTB-Pad19)
- U4 pad 2: Net-(U4-DIG_0) -> Net-(U4-GPB1)
- U4 pad 20: Net-(U4-SEG_C) -> unconnected-(U4-INTA-Pad20)
- U4 pad 23: Net-(U4-SEG_D) -> unconnected-(U4-GPA2-Pad23)
- U4 pad 3: unconnected-(U4-DIG_4-Pad3) -> Net-(U4-GPB2)
- U4 pad 4: GND -> Net-(U4-GPB3)
- U4 pad 5: unconnected-(U4-DIG_6-Pad5) -> Net-(U4-GPB4)
- U4 pad 6: unconnected-(U4-DIG_2-Pad6) -> Net-(U4-GPB5)
- U4 pad 7: unconnected-(U4-DIG_3-Pad7) -> Net-(SW9-A)
- U4 pad 8: unconnected-(U4-DIG_7-Pad8) -> Net-(SW9-B)
- U4 pad 9: GND -> +5V
- U6 pad 1: /buttons/COM -> Net-(U4-GPB1)
- U6 pad 10: /buttons/S0 -> Net-(U6-DIG_5)
- U6 pad 11: /buttons/S1 -> Net-(U6-DIG_1)
- U6 pad 12: GND -> unconnected-(U6-LOAD-Pad12)
- U6 pad 13: /buttons/S3 -> Net-(U4-GPB0)
- U6 pad 14: /buttons/S2 -> Net-(U6-SEG_A)
- U6 pad 15: GND -> Net-(U6-SEG_F)
- U6 pad 16: Net-(U6-I15) -> Net-(U6-SEG_B)
- U6 pad 18: Net-(U6-I13) -> unconnected-(U6-ISET-Pad18)
- U6 pad 19: Net-(U6-I12) -> +5V
- U6 pad 23: Net-(U6-I8) -> Net-(U6-SEG_D)
- U6 pad 24: +5V -> unconnected-(U6-DOUT-Pad24)
- U6 pad 4: Net-(U6-I5) -> Earth
- U6 pad 5: Net-(U6-I4) -> Net-(U6-DIG_6)
- U6 pad 8: Net-(U6-I1) -> unconnected-(U6-DIG_7-Pad8)
- U6 pad 9: Net-(U6-I0) -> Earth
- solo1 pad 1: Net-(U6-I0) -> +5V
- solo1 pad 2: GND -> Net-(U4-GPB4)
- solo1 pad 3: Net-(U4-SEG_A) -> Net-(U6-DIG_6)
- solo1 pad 4: Net-(U4-DIG_1) -> Net-(U6-SEG_B)
- solo2 pad 1: Net-(U6-I1) -> +5V
- solo2 pad 2: GND -> Net-(U4-GPB5)
- solo2 pad 3: Net-(U4-SEG_B) -> Net-(U6-DIG_6)
- solo2 pad 4: Net-(U4-DIG_1) -> Net-(U6-SEG_D)
Routing:
- net GND: track 934.2 -> 0.00 mm
- net Net-(U11-SEG_A): track 822.3 -> 0.00 mm, vias 8 -> 0
- net Net-(U11-SEG_B): track 800.4 -> 0.00 mm, vias 8 -> 0
- net Net-(U11-SEG_C): track 784.8 -> 0.00 mm, vias 8 -> 0
- net Net-(U11-SEG_D): track 763.7 -> 0.00 mm, vias 8 -> 0
- net Net-(U11-SEG_E): track 738.8 -> 0.00 mm, vias 8 -> 0
- net Net-(U12-SEG_A): track 679.6 -> 0.00 mm, vias 8 -> 0
- net Net-(U12-SEG_B): track 659.0 -> 0.00 mm, vias 8 -> 0
- net Net-(U12-SEG_C): track 644.0 -> 0.00 mm, vias 8 -> 0
- net Net-(U12-SEG_D): track 623.5 -> 0.00 mm, vias 8 -> 0
- net Net-(U12-SEG_E): track 599.5 -> 0.00 mm, vias 8 -> 0
- net Net-(U9-SEG_A): track 596.9 -> 0.00 mm, vias 8 -> 0
- net Net-(U9-SEG_B): track 572.4 -> 0.00 mm, vias 8 -> 0
- net Net-(U9-SEG_C): track 542.8 -> 0.00 mm, vias 8 -> 0
- net Net-(U9-SEG_D): track 516.3 -> 0.00 mm, vias 8 -> 0
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